File: usb_typec_serial_insulation_adum121n/usb_typec_serial_insulation.kicad_sch (KiCad schematic)
At the start: 3 parts, among them J1 Conn_01x06_Socket, J2 Conn_01x06_Socket, U1 ADuM121N

Commit message: add C1, C2 adum121N V1.1
add C1, C2 adum121N V1.1
Parts:
- added C1, C2: 0.1uF,10V(=5V*2), Capacitor_SMD:C_0603_1608Metric_Pad1.08x0.95mm_HandSolder, symbol Device:C
Connections:
- net GND1: now also C1.2
- net GND2: now also C2.2
- net VCC1: now also C1.1
- net VCC2: now also C2.1
Changed lines of the file:
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@@
 	(title_block
 		(title "usb_typec_serial_insulation")
-		(date "2026-02-11")
-		(rev "V1")
+		(date "2026-02-12")
+		(rev "V1.1")
 		(company "takurx")
 		(comment 1 "ADuM121N")
+		(comment 2 "add C1, C2")
 	)
 	(text "1 RTS\n2 RXD\n3 TXD\n4 VCC\n5 CTS\n6 GND"
@@
 	(wire
 		(pts
+			(xy 111.76 107.95) (xy 118.11 107.95)
+		)
+		(stroke
+			(width 0)
+			(type default)
+		)
+	)
+	(wire
+		(pts
 			(xy 118.11 78.74) (xy 118.11 93.98)
 		)
@@
 	(wire
 		(pts
+			(xy 111.76 86.36) (xy 111.76 107.95)
+		)
+		(stroke
+			(width 0)
+			(type default)
+		)
+	)
+	(wire
+		(pts
+			(xy 168.91 107.95) (xy 161.29 107.95)
+		)
+		(stroke
+			(width 0)
+			(type default)
+		)
+	)
+	(wire
+		(pts
+			(xy 168.91 86.36) (xy 168.91 107.95)
+		)
+		(stroke
+			(width 0)
+			(type default)
+		)
+	)
+	(wire
+		(pts
+			(xy 111.76 78.74) (xy 118.11 78.74)
+		)
+		(stroke
+			(width 0)
+			(type default)
+		)
+	)
+	(wire
+		(pts
 			(xy 107.95 96.52) (xy 128.27 96.52)
 		)
@@
 		(pts
 			(xy 118.11 107.95) (xy 118.11 99.06)
+		)
+		(stroke
+			(width 0)
+			(type default)
+		)
+	)
+	(wire
+		(pts
+			(xy 163.83 78.74) (xy 168.91 78.74)
 		)
 		(stroke
@@
 	)
 	(symbol
+		(lib_id "Device:C")
+		(at 168.91 82.55 0)
+		(unit 1)
+		(exclude_from_sim no)
+		(in_bom yes)
+		(on_board yes)
+		(dnp no)
+		(fields_autoplaced yes)
+		(property "Reference" "C1"
+			(at 172.72 81.2799 0)
+			(effects
+				(font
+					(size 1.27 1.27)
+				)
+				(justify left)
+			)
+		)
+		(property "Value" "0.1uF,10V(=5V*2)"
+			(at 172.72 83.8199 0)
+			(effects
+				(font
+					(size 1.27 1.27)
+				)
+				(justify left)
+			)
+		)
+		(property "Footprint" "Capacitor_SMD:C_0603_1608Metric_Pad1.08x0.95mm_HandSolder"
+			(at 169.8752 86.36 0)
+			(effects
+				(font
+					(size 1.27 1.27)
+				)
+				(hide yes)
+			)
+		)
+		(property "Datasheet" "~"
+			(at 168.91 82.55 0)
+			(effects
+				(font
+					(size 1.27 1.27)
+				)
+				(hide yes)
+			)
+		)
+		(property "Description" "Unpolarized capacitor"
+			(at 168.91 82.55 0)
+			(effects
+				(font
+					(size 1.27 1.27)
+				)
+				(hide yes)
+			)
+		)
+		(pin "2"
+		)
+		(pin "1"
+		)
+		(instances
+			(project ""
+				(path "/09755bd0-05d9-43ff-a82a-95a2569aaa80"
+					(reference "C1")
+					(unit 1)
+				)
+			)
+		)
+	)
+	(symbol
 		(lib_id "power:VCC")
 		(at 163.83 72.39 0)
@@
 					(unit 1)
 				)
+			)
+		)
+	)
+	(symbol
+		(lib_id "Device:C")
+		(at 111.76 82.55 0)
+		(unit 1)
+		(exclude_from_sim no)
+		(in_bom yes)
+		(on_board yes)
+		(dnp no)
+		(fields_autoplaced yes)
+		(property "Reference" "C2"
+			(at 115.57 81.2799 0)
+			(effects
+				(font
+					(size 1.27 1.27)
+				)
+				(justify left)
+			)
+		)
+		(property "Value" "0.1uF,10V(=5V*2)"
+			(at 115.57 83.8199 0)
+			(effects
+				(font
+					(size 1.27 1.27)
+				)
+				(justify left)
+			)
+		)
+		(property "Footprint" "Capacitor_SMD:C_0603_1608Metric_Pad1.08x0.95mm_HandSolder"
+			(at 112.7252 86.36 0)
+			(effects
+				(font
+					(size 1.27 1.27)
+				)
+				(hide yes)
+			)
+		)
+		(property "Datasheet" "~"
+			(at 111.76 82.55 0)
+			(effects
+				(font
+					(size 1.27 1.27)
+				)
+				(hide yes)
+			)
+		)
+		(property "Description" "Unpolarized capacitor"
+			(at 111.76 82.55 0)
+			(effects
+				(font
+					(size 1.27 1.27)
+				)
+				(hide yes)
+			)
+		)
+		(pin "1"
+		)
+		(pin "2"
+		)
+		(instances
+			(project ""
+				(path "/09755bd0-05d9-43ff-a82a-95a2569aaa80"
+					(reference "C2")
+					(unit 1)
+				)

Commit message: add 1412 other plan
add 1412 other plan
Other:
- note added: "Arduino 1 NC 2 TX 3 RX 4 VCC 5 NC 6 GND"
Changed lines of the file:
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@@
+		)
+	)
+	(text "Arduino\n1 NC\n2 TX\n3 RX\n4 VCC\n5 NC\n6 GND"
+		(exclude_from_sim no)
+		(at 221.234 102.362 0)
+		(effects
+			(font
+				(size 1.27 1.27)
+			)
+			(justify left)
 		)
 	)

Commit message: modify 121N, V2.0
modify 121N, V2.0
Connections:
- net at U1.2 (VOA): now also J1.2 (Pin_2); no longer J1.3 (Pin_3)
- net at U1.3 (VIB): now also J1.3 (Pin_3); no longer J1.2 (Pin_2)
Other:
- note added: "1 NC 2 VOA, TXD -> 3 VIB, RXD <- 4 VCC 5 NC 6 GND"
- note added: "1 NC 2 VOB, TXD <- 3 VIA, RXD -> 4 VCC 5 NC 6 GND"
- note added: "1 RTS -> 2 RXD <- 3 TXD -> 4 VCC 5 CTS <- 6 GND"
- note added: "1 RTS <- 2 RXD -> 3 TXD <- 4 VCC 5 CTS -> 6 GND"
- note added: "Arduino 1 NC/RTS -> 2 RXD <- 3 TXD -> 4 VCC 5 NC/CTS <- 6 GND"
- note added: "ArduinoのUART入出力が接続される場合"
- note added: "J1, J2のピン配置は、 ポカヨケで秋月電子のCH340Eモジュールがどちら側でも付けれるように合わせる Arduinoの場合はArduino側を合わせる"
- note removed: "1 RTS 2 RXD 3 TXD 4 VCC 5 CTS 6 GND"
- note removed: "Arduino 1 NC 2 TX 3 RX 4 VCC 5 NC 6 GND"
- note removed: "ArduinoのUART出力などが接続されることを想定する"
Changed lines of the file:
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@@
 	(title_block
 		(title "usb_typec_serial_insulation")
-		(date "2026-02-12")
-		(rev "V1.1")
+		(date "2026-03-26")
+		(rev "V2.0")
 		(company "takurx")
 		(comment 1 "ADuM121N")
 		(comment 2 "add C1, C2")
-	)
-	(text "1 RTS\n2 RXD\n3 TXD\n4 VCC\n5 CTS\n6 GND"
-		(exclude_from_sim no)
-		(at 199.39 103.378 0)
-		(effects
-			(font
-				(size 1.27 1.27)
-			)
-		)
-	)
-	(text "ArduinoのUART出力などが接続されることを想定する\n"
-		(exclude_from_sim no)
-		(at 215.392 71.374 90)
+		(comment 3 "modify pinout 2, 3")
+	)
+	(text "1 NC\n2 VOA, TXD ->\n3 VIB, RXD <-\n4 VCC\n5 NC\n6 GND"
+		(exclude_from_sim no)
+		(at 194.31 104.648 0)
+		(effects
+			(font
+				(size 1.27 1.27)
+			)
+			(justify left)
+		)
+	)
+	(text "ArduinoのUART入出力が接続される場合"
+		(exclude_from_sim no)
+		(at 25.146 74.422 90)
 		(effects
 			(font
@@
 	(text "秋月電子のCH340E USBシリアル変換モジュールを接続することを想定する\nCH340E USBシリアル変換モジュール Type-C: 半導体 秋月電子通商-電子部品・ネット通販\nhttps://akizukidenshi.com/catalog/g/g114745/"
 		(exclude_from_sim no)
-		(at 70.612 63.5 90)
+		(at 229.362 56.642 90)
 		(effects
 			(font
@@
 		)
 	)
-	(text "1 RTS\n2 RXD\n3 TXD\n4 VCC\n5 CTS\n6 GND"
-		(exclude_from_sim no)
-		(at 88.9 106.68 0)
-		(effects
-			(font
-				(size 1.27 1.27)
-			)
-		)
-	)
-	(text "Arduino\n1 NC\n2 TX\n3 RX\n4 VCC\n5 NC\n6 GND"
-		(exclude_from_sim no)
-		(at 221.234 102.362 0)
-		(effects
-			(font
-				(size 1.27 1.27)
-			)
-			(justify left)
+	(text "1 NC\n2 VOB, TXD <-\n3 VIA, RXD ->\n4 VCC\n5 NC\n6 GND"
+		(exclude_from_sim no)
+		(at 83.82 106.172 0)
+		(effects
+			(font
+				(size 1.27 1.27)
+			)
+			(justify left)
+		)
+	)
+	(text "1 RTS <-\n2 RXD ->\n3 TXD <-\n4 VCC\n5 CTS ->\n6 GND"
+		(exclude_from_sim no)
+		(at 214.376 104.648 0)
+		(effects
+			(font
+				(size 1.27 1.27)
+			)
+			(justify left)
+		)
+	)
+	(text "1 RTS ->\n2 RXD <-\n3 TXD ->\n4 VCC\n5 CTS <-\n6 GND"
+		(exclude_from_sim no)
+		(at 63.5 106.172 0)
+		(effects
+			(font
+				(size 1.27 1.27)
+			)
+			(justify left)
+		)
+	)
+	(text "Arduino\n1 NC/RTS ->\n2 RXD <-\n3 TXD ->\n4 VCC\n5 NC/CTS <-\n6 GND"
+		(exclude_from_sim no)
+		(at 30.988 105.41 0)
+		(effects
+			(font
+				(size 1.27 1.27)
+			)
+			(justify left)
+		)
+	)
+	(text "J1, J2のピン配置は、\nポカヨケで秋月電子のCH340Eモジュールがどちら側でも付けれるように合わせる\nArduinoの場合はArduino側を合わせる"
+		(exclude_from_sim no)
+		(at 111.252 130.302 0)
+		(effects
+			(font
+				(size 1.27 1.27)
+			)
+			(justify left)
+		)
+	)
+	(text "秋月電子のCH340E USBシリアル変換モジュールを接続することを想定する\nCH340E USBシリアル変換モジュール Type-C: 半導体 秋月電子通商-電子部品・ネット通販\nhttps://akizukidenshi.com/catalog/g/g114745/"
+		(exclude_from_sim no)
+		(at 58.166 56.388 90)
+		(effects
+			(font
+				(size 1.27 1.27)
+			)
+			(justify right)
 		)
 	)
@@
 	(wire
 		(pts
+			(xy 185.42 91.44) (xy 161.29 91.44)
+		)
+		(stroke
+			(width 0)
+			(type default)
+		)
+	)
+	(wire
+		(pts
 			(xy 118.11 114.3) (xy 118.11 107.95)
 		)
@@
 	(wire
 		(pts
+			(xy 161.29 96.52) (xy 153.67 96.52)
+		)
+		(stroke
+			(width 0)
+			(type default)
+		)
+	)
+	(wire
+		(pts
 			(xy 111.76 107.95) (xy 118.11 107.95)
 		)
@@
 	(wire
 		(pts
+			(xy 102.87 91.44) (xy 128.27 91.44)
+		)
+		(stroke
+			(width 0)
+			(type default)
+		)
+	)
+	(wire
+		(pts
 			(xy 111.76 86.36) (xy 111.76 107.95)
 		)
@@
 	(wire
 		(pts
-			(xy 107.95 96.52) (xy 128.27 96.52)
-		)
-		(stroke
-			(width 0)
-			(type default)
-		)
-	)
-	(wire
-		(pts
 			(xy 138.43 104.14) (xy 138.43 107.95)
 		)
@@
 	(wire
 		(pts
+			(xy 114.3 88.9) (xy 102.87 88.9)
+		)
+		(stroke
+			(width 0)
+			(type default)
+		)
+	)
+	(wire
+		(pts
 			(xy 143.51 107.95) (xy 161.29 107.95)
 		)
@@
 	(wire
 		(pts
-			(xy 172.72 88.9) (xy 172.72 96.52)
-		)
-		(stroke
-			(width 0)
-			(type default)
-		)
-	)
-	(wire
-		(pts
-			(xy 107.95 96.52) (xy 107.95 88.9)
+			(xy 158.75 88.9) (xy 158.75 91.44)
+		)
+		(stroke
+			(width 0)
+			(type default)
+		)
+	)
+	(wire
+		(pts
+			(xy 158.75 91.44) (xy 153.67 91.44)
 		)
 		(stroke
@@
 	(wire
 		(pts
-			(xy 153.67 91.44) (xy 185.42 91.44)
-		)
-		(stroke
-			(width 0)
-			(type default)
-		)
-	)
-	(wire
-		(pts
-			(xy 172.72 96.52) (xy 153.67 96.52)
-		)
-		(stroke
-			(width 0)
-			(type default)
-		)
-	)
-	(wire
-		(pts
 			(xy 138.43 107.95) (xy 118.11 107.95)
 		)
@@
 	(wire
 		(pts
-			(xy 185.42 88.9) (xy 172.72 88.9)
-		)
-		(stroke
-			(width 0)
-			(type default)
-		)
-	)
-	(wire
-		(pts
 			(xy 185.42 93.98) (xy 163.83 93.98)
 		)
@@
 	(wire
 		(pts
+			(xy 185.42 88.9) (xy 158.75 88.9)
+		)
+		(stroke
+			(width 0)
+			(type default)
+		)
+	)
+	(wire
+		(pts
 			(xy 138.43 78.74) (xy 118.11 78.74)
 		)
@@
 	(wire
 		(pts
-			(xy 102.87 91.44) (xy 128.27 91.44)
-		)
-		(stroke
-			(width 0)
-			(type default)
-		)
-	)
-	(wire
-		(pts
-			(xy 107.95 88.9) (xy 102.87 88.9)
-		)
-		(stroke
+			(xy 161.29 91.44) (xy 161.29 96.52)
+		)
+		(stroke
+			(width 0)
+			(type default)
+		)
+	)
+	(wire
+		(pts
+			(xy 128.27 96.52) (xy 114.3 96.52)
+		)
+		(stroke
+			(width 0)
+			(type default)
+		)
+	)
+	(wire
+		(pts
+			(xy 114.3 96.52) (xy 114.3 88.9)
+		)
+		(stroke
