File: usb_typec_serial_insulation_adum121n/usb_typec_serial_insulation.kicad_pcb (KiCad board)
At the start: 2 copper layers, 20 x 17 mm, 5 parts, among them J1 Conn_01x06_Socket, J2 Conn_01x06_Socket, U1 ADuM121N

Commit message: add rev3.0 zebra 121N
add rev3.0 zebra 121N
Other:
- board text added: "ZEBRA ADuM121N USB SERIAL ISOLATOR REV 3.0 260911 TSUKUSEI WORKS"
- board text removed: "usb typec serial inslation ADuM121N V2.1 260430 takurx"
Changed lines of the file:
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@@
 		)
 	)
-	(gr_text "usb typec serial inslation\nADuM121N\nV2.1 260430 takurx"
-		(at 139.6 89.7 90)
+	(gr_text "ZEBRA ADuM121N\nUSB SERIAL ISOLATOR\nREV 3.0 260911\nTSUKUSEI WORKS"
+		(at 140.5 90 90)
 		(layer "B.SilkS")
 		(effects
