File: usb_typec_serial_insulation_adum1412/usb_typec_serial_insulation_adum1412.kicad_sch (KiCad schematic)
At the start: 5 parts, among them J1 Conn_01x06_Socket, J2 Conn_01x06_Socket, U1 ADuM1412

Commit message: modify 1412
modify 1412
Connections:
- net at U1.3 (VIA): now also J1.3 (Pin_3); no longer J1.2 (Pin_2)
- net at U1.4 (VIB): now also J1.1 (Pin_1); no longer J1.5 (Pin_5)
- net at U1.5 (VOC): now also J1.2 (Pin_2); no longer J1.3 (Pin_3)
- net at U1.6 (VOD): now also J1.5 (Pin_5); no longer J1.1 (Pin_1)
Other:
- note added: "1 RTS <- 2 RXD -> 3 TXD <- 4 VCC 5 CTS -> 6 GND"
- note added: "1 VIB, RTS <- 2 VOC, RXD -> 3 VIA, TXD <- 4 VCC 5 VOD, CTS -> 6 GND"
- note added: "1 VID, RTS -> 2 VOA, RXD <- 3 VIC, TXD -> 4 VCC 5 VOB, CTS <- 6 GND"
- note added: "Arduino 1 RTS -> 2 RXD <- 3 TXD -> 4 VCC 5 CTS <- 6 GND"
- note added: "J1, J2のピン配置は、 ポカヨケで秋月電子のCH340Eモジュールがどちら側でも付けれるように合わせる Arduinoの場合はArduino側を合わせる"
- note removed: "Arduino 1 CTS -> 2 TX <- 3 RX -> 4 VCC 5 RTS <- 6 GND"
