File: usb_typec_serial_insulation_adum1412/usb_typec_serial_insulation_adum1412.kicad_pcb (KiCad board)
At the start: 2 copper layers, 27 x 17 mm, 5 parts, among them J1 Conn_01x06_Socket, J2 Conn_01x06_Socket, U1 ADuM1412

Commit message: modify 1412
modify 1412
Connections:
- U1 pad 3: Net-(J1-Pin_2) -> Net-(J1-Pin_3)
- U1 pad 4: Net-(J1-Pin_5) -> Net-(J1-Pin_1)
- U1 pad 5: Net-(J1-Pin_3) -> Net-(J1-Pin_2)
- U1 pad 6: Net-(J1-Pin_1) -> Net-(J1-Pin_5)
Routing:
- net Net-(J1-Pin_1): track 8.08 -> 11.9 mm, vias 0 -> 2
- net Net-(J1-Pin_5): track 7.78 -> 11.0 mm, vias 0 -> 2
- net Net-(J1-Pin_2): track 9.37 -> 8.11 mm, vias 2 -> 0
- net Net-(J1-Pin_3): track 6.50 -> 7.56 mm
Other:
- board text added: "usb typec serial inslation ADuM1412 V3.0 260326 takurx"
- board text removed: "usb typec serial inslation ADuM1412 V2.0 260212 takurx"
Changed lines of the file:
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@@
 	(title_block
 		(title "usb typec serial insulation")
-		(date "2026-02-12")
-		(rev "V2.0")
+		(date "2026-03-26")
+		(rev "V3.0")
 		(company "takurx")
 		(comment 1 "ADuM1412")
+		(comment 2 "modify pinout 1,2,3,5")
 	)
 	(layers
@@
 			(layers "F.Cu" "F.Mask" "F.Paste")
 			(roundrect_rratio 0.25)
-			(net 3 "Net-(J1-Pin_2)")
+			(net 2 "Net-(J1-Pin_3)")
 			(pinfunction "VIA")
 			(pintype "input")
@@
 			(layers "F.Cu" "F.Mask" "F.Paste")
 			(roundrect_rratio 0.25)
-			(net 4 "Net-(J1-Pin_5)")
+			(net 5 "Net-(J1-Pin_1)")
 			(pinfunction "VIB")
 			(pintype "input")
@@
 			(layers "F.Cu" "F.Mask" "F.Paste")
 			(roundrect_rratio 0.25)
-			(net 2 "Net-(J1-Pin_3)")
+			(net 3 "Net-(J1-Pin_2)")
 			(pinfunction "VOC")
 			(pintype "output")
@@
 			(layers "F.Cu" "F.Mask" "F.Paste")
 			(roundrect_rratio 0.25)
-			(net 5 "Net-(J1-Pin_1)")
+			(net 4 "Net-(J1-Pin_5)")
 			(pinfunction "VOD")
 			(pintype "output")
@@
 		)
 	)
-	(gr_text "usb typec serial inslation\nADuM1412\nV2.0 260212 takurx"
+	(gr_text "usb typec serial inslation\nADuM1412\nV3.0 260326 takurx"
 		(at 150.3 89.6 90)
 		(layer "B.SilkS")
@@
 	)
 	(segment
-		(start 152.135 96.365)
-		(end 152.5 96)
+		(start 149.595 98.905)
+		(end 146.15 98.905)
 		(width 0.6)
 		(layer "F.Cu")
@@
 	)
 	(segment
-		(start 146.15 96.365)
-		(end 152.135 96.365)
+		(start 146.155 98.9)
+		(end 146.15 98.905)
 		(width 0.6)
 		(layer "F.Cu")
@@
 	)
 	(segment
-		(start 147.8 98.9)
-		(end 146.155 98.9)
-		(width 0.6)
-		(layer "F.Cu")
-		(net 3)
-	)
-	(segment
-		(start 151.94 93.46)
-		(end 150.1 95.3)
+		(start 152.5 96)
+		(end 149.595 98.905)
+		(width 0.6)
+		(layer "F.Cu")
+		(net 2)
+	)
+	(segment
+		(start 152.5 93.46)
+		(end 149.595 96.365)
 		(width 0.6)
 		(layer "F.Cu")
@@
 	)
 	(segment
-		(start 146.155 98.9)
-		(end 146.15 98.905)
+		(start 149.595 96.365)
+		(end 146.15 96.365)
 		(width 0.6)
 		(layer "F.Cu")
 		(net 3)
 	)
+	(segment
+		(start 146.230686 95.014314)
+		(end 146.15 95.095)
+		(width 0.6)
+		(layer "F.Cu")
+		(net 4)
+	)
+	(segment
+		(start 152.32778 101.08)
+		(end 150.439576 99.191796)
+		(width 0.6)
+		(layer "F.Cu")
+		(net 4)
+	)
+	(segment
+		(start 152.5 101.08)
+		(end 152.32778 101.08)
+		(width 0.6)
+		(layer "F.Cu")
+		(net 4)
+	)
+	(segment
+		(start 149.814314 95.014314)
+		(end 146.230686 95.014314)
+		(width 0.6)
+		(layer "F.Cu")
+		(net 4)
+	)
 	(via
-		(at 147.8 98.9)
+		(at 150.439576 99.191796)
 		(size 0.6)
 		(drill 0.3)
 		(layers "F.Cu" "B.Cu")
-		(net 3)
+		(net 4)
 	)
 	(via
-		(at 150.1 95.3)
+		(at 149.814314 95.014314)
 		(size 0.6)
 		(drill 0.3)
 		(layers "F.Cu" "B.Cu")
-		(net 3)
-	)
-	(segment
-		(start 150.1 96.6)
-		(end 147.8 98.9)
+		(net 4)
+	)
+	(segment
+		(start 149.814314 98.566534)
+		(end 149.814314 95.014314)
 		(width 0.6)
 		(layer "B.Cu")
-		(net 3)
-	)
-	(segment
-		(start 150.1 95.3)
-		(end 150.1 96.6)
+		(net 4)
+	)
+	(segment
+		(start 150.439576 99.191796)
+		(end 149.814314 98.566534)
 		(width 0.6)
 		(layer "B.Cu")
-		(net 3)
-	)
-	(segment
-		(start 146.15 97.635)
-		(end 149.055 97.635)
-		(width 0.6)
-		(layer "F.Cu")
 		(net 4)
 	)
 	(segment
-		(start 149.055 97.635)
-		(end 152.5 101.08)
-		(width 0.6)
-		(layer "F.Cu")
-		(net 4)
-	)
-	(segment
-		(start 148.325 95.095)
-		(end 152.5 90.92)
+		(start 149 92.9)
+		(end 148.8 92.9)
 		(width 0.6)
 		(layer "F.Cu")
@@
 	)
 	(segment
-		(start 146.15 95.095)
-		(end 148.325 95.095)
-		(width 0.6)
-		(layer "F.Cu")
+		(start 146.185 97.6)
+		(end 146.15 97.635)
+		(width 0.6)
+		(layer "F.Cu")
+		(net 5)
+	)
+	(segment
+		(start 148.8 97.6)
+		(end 146.185 97.6)
+		(width 0.6)
+		(layer "F.Cu")
+		(net 5)
+	)
+	(segment
+		(start 152.5 90.92)
+		(end 150.98 90.92)
+		(width 0.6)
+		(layer "F.Cu")
+		(net 5)
+	)
+	(segment
+		(start 150.98 90.92)
+		(end 149 92.9)
+		(width 0.6)
+		(layer "F.Cu")
+		(net 5)
+	)
+	(via
+		(at 148.8 97.6)
+		(size 0.6)
+		(drill 0.3)
+		(layers "F.Cu" "B.Cu")
+		(net 5)
+	)
+	(via
+		(at 148.8 92.9)
+		(size 0.6)
+		(drill 0.3)
+		(layers "F.Cu" "B.Cu")
+		(net 5)
+	)
+	(segment
+		(start 148.8 92.9)
+		(end 148.8 97.6)
+		(width 0.6)
+		(layer "B.Cu")
 		(net 5)
 	)
@@
 	)
 	(segment
-		(start 146.175 93.8)
-		(end 146.15 93.825)
-		(width 0.6)
-		(layer "F.Cu")
-		(net 9)
-	)
-	(segment
 		(start 146.15 101.445)
 		(end 147.755 101.445)
@@
 	)
 	(segment
+		(start 146.15 93.825)
+		(end 150.925 93.825)
+		(width 0.6)
+		(layer "F.Cu")
+		(net 9)
+	)
+	(segment
 		(start 147.755 101.445)
 		(end 147.8 101.4)
@@
 	)
 	(segment
-		(start 147.8 93.8)
-		(end 146.175 93.8)
-		(width 0.6)
-		(layer "F.Cu")
-		(net 9)
-	)
-	(segment
 		(start 146.1375 104.1)
 		(end 146.1375 101.4575)
+		(width 0.6)
+		(layer "F.Cu")
+		(net 9)
+	)
+	(segment
+		(start 150.925 93.825)
+		(end 150.964314 93.864314)
 		(width 0.6)
 		(layer "F.Cu")
@@
 	)
 	(via
-		(at 147.8 93.8)
+		(at 150.964314 93.864314)
 		(size 0.6)
 		(drill 0.3)
@@
 	)
 	(segment
-		(start 151 93.9)
-		(end 147.9 93.9)
-		(width 0.6)
-		(layer "B.Cu")
-		(net 9)
-	)
-	(segment
 		(start 147.8 101.4)
 		(end 149.64 101.4)
 		(width 0.6)
 		(layer "B.Cu")
-		(net 9)
-	)
-	(segment
-		(start 147.9 93.9)
-		(end 147.8 93.8)
-		(width 0.6)
-		(layer "B.Cu")

Commit message: add silk description
add silk description
Other:
- board text added: "-> CTS VOD"
- board text added: "-> RTS VID"
- board text added: "-> RX1 VOC"
- board text added: "-> TX2 VIC"
- board text added: "<- CTS VOB"
- board text added: "<- RTS VIB"
- board text added: "<- RX2 VOA"
- board text added: "<- TX1 VIA"
- board text added: "usb typec serial inslation ADuM1412 V3.1 260326 takurx"
- board text removed: "CTS"
- board text removed: "RTS"
- board text removed: "RX1"
- board text removed: "RX2"
- board text removed: "TX1"
- board text removed: "TX2"
- board text removed: "usb typec serial inslation ADuM1412 V3.0 260326 takurx"
Changed lines of the file:
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@@
 		(title "usb typec serial insulation")
 		(date "2026-03-26")
-		(rev "V3.0")
+		(rev "V3.1")
 		(company "takurx")
 		(comment 1 "ADuM1412")
@@
 	)
 	(gr_text "VCC2"
-		(at 132.1 99 0)
+		(at 132.4 99 0)
 		(layer "F.SilkS")
 		(effects
@@
 	)
 	(gr_text "GND2"
-		(at 132.1 103.2 0)
+		(at 132.2 103.2 0)
 		(layer "F.SilkS")
 		(effects
@@
 		)
 	)
-	(gr_text "RX2"
-		(at 132.1 93.5 0)
+	(gr_text "<-\nRX2\nVOA"
+		(at 132.4 94.7 0)
 		(layer "F.SilkS")
 		(effects
@@
 		)
 	)
-	(gr_text "TX2"
-		(at 132.1 96.5 0)
+	(gr_text "->\nTX2\nVIC"
+		(at 132.4 97.4 0)
 		(layer "F.SilkS")
 		(effects
@@
 	)
 	(gr_text "VCC1"
-		(at 148.7 99.1 0)
+		(at 148.4 99.1 0)
 		(layer "F.SilkS")
 		(effects
@@
 		)
 	)
-	(gr_text "TX1"
-		(at 149.4 96.5 0)
+	(gr_text "<-\nTX1\nVIA"
+		(at 149 97.7 0)
 		(layer "F.SilkS")
 		(effects
@@
 		)
 	)
-	(gr_text "RTS"
-		(at 132.1 91 0)
+	(gr_text "->\nRTS\nVID"
+		(at 132.4 91.9 0)
 		(layer "F.SilkS")
 		(effects
@@
 		)
 	)
-	(gr_text "RX1"
-		(at 149.2 93.9 0)
+	(gr_text "->\nRX1\nVOC"
+		(at 148.9 94.9 0)
 		(layer "F.SilkS")
 		(effects
@@
 		)
 	)
-	(gr_text "CTS"
-		(at 132.2 101.5 0)
+	(gr_text "<-\nCTS\nVOB"
+		(at 132.4 102.1 0)
 		(layer "F.SilkS")
 		(effects
@@
 		)
 	)
-	(gr_text "RTS"
-		(at 149.2 91.3 0)
+	(gr_text "<-\nRTS\nVIB"
+		(at 149 92 0)
 		(layer "F.SilkS")
 		(effects
@@
 		)
 	)
-	(gr_text "CTS"
-		(at 149.2 101.5 0)
+	(gr_text "->\nCTS\nVOD"
+		(at 148.9 102.3 0)
 		(layer "F.SilkS")
 		(effects
@@
 		)
 	)
-	(gr_text "usb typec serial inslation\nADuM1412\nV3.0 260326 takurx"
+	(gr_text "usb typec serial inslation\nADuM1412\nV3.1 260326 takurx"
 		(at 150.3 89.6 90)
 		(layer "B.SilkS")

Commit message: add pinout description
add pinout description
Other:
- board text added: "-> CTS VOB"
- board text added: "-> RTS VIB"
- board text added: "-> RX2 VOA"
- board text added: "-> TX1 VIA"
- board text added: "<- CTS VOD"
- board text added: "<- RTS VID"
- board text added: "<- RX1 VOC"
- board text added: "<- TX2 VIC"
- board text added: "usb typec serial inslation ADuM1412 V3.2 260430 takurx"
- board text removed: "usb typec serial inslation ADuM1412 V3.1 260326 takurx"
Changed lines of the file:
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@@
 	(title_block
 		(title "usb typec serial insulation")
-		(date "2026-03-26")
-		(rev "V3.1")
+		(date "2026-04-30")
+		(rev "V3.2")
 		(company "takurx")
 		(comment 1 "ADuM1412")
 		(comment 2 "modify pinout 1,2,3,5")
+		(comment 3 "add pinout description, B.Silk")
 	)
 	(layers
@@
 		)
 	)
-	(gr_text "usb typec serial inslation\nADuM1412\nV3.1 260326 takurx"
-		(at 150.3 89.6 90)
+	(gr_text "->\nRTS\nVIB"
+		(at 150.205 92 0)
+		(layer "B.SilkS")
+		(effects
+			(font
+				(size 0.6 0.6)
+				(thickness 0.075)
+			)
+			(justify left bottom mirror)
+		)
+	)
+	(gr_text "usb typec serial inslation\nADuM1412\nV3.2 260430 takurx"
+		(at 143.1 89.6 90)
 		(layer "B.SilkS")
 		(effects
@@
 			)
 			(justify left bottom mirror)
+		)
+	)
+	(gr_text "->\nRX2\nVOA"
+		(at 134.3 95 0)
+		(layer "B.SilkS")
+		(effects
+			(font
+				(size 0.6 0.6)
+				(thickness 0.075)
+			)
+			(justify left bottom mirror)
+		)
+	)
+	(gr_text "GND2"
+		(at 134.9 104.1 -0)
+		(layer "B.SilkS")
+		(effects
+			(font
+				(size 0.6 0.6)
+				(thickness 0.075)
+			)
+			(justify left bottom mirror)
+		)
+	)
+	(gr_text "->\nTX1\nVIA"
+		(at 150.205 97.7 0)
+		(layer "B.SilkS")
+		(effects
+			(font
+				(size 0.6 0.6)
+				(thickness 0.075)
+			)
+			(justify left bottom mirror)
+		)
+	)
+	(gr_text "->\nCTS\nVOB"
+		(at 134.3 102.2 0)
+		(layer "B.SilkS")
+		(effects
+			(font
+				(size 0.6 0.6)
+				(thickness 0.075)
+			)
+			(justify left bottom mirror)
+		)
+	)
+	(gr_text "<-\nTX2\nVIC"
+		(at 134.3 98 0)
+		(layer "B.SilkS")
+		(effects
+			(font
+				(size 0.6 0.6)
+				(thickness 0.075)
+			)
+			(justify left bottom mirror)
+		)
+	)
+	(gr_text "<-\nCTS\nVOD"
+		(at 150.305 102.3 0)
+		(layer "B.SilkS")
+		(effects
+			(font
+				(size 0.6 0.6)
+				(thickness 0.075)
+			)
+			(justify left bottom mirror)
+		)
+	)
+	(gr_text "VCC1"
+		(at 150.3 99.1 -0)
+		(layer "B.SilkS")
+		(effects
+			(font
+				(size 0.6 0.6)
+				(thickness 0.075)
+			)
+			(justify left bottom mirror)
+		)
+	)
+	(gr_text "GND1"
+		(at 150.4 104.2 -0)
+		(layer "B.SilkS")
+		(effects
+			(font
+				(size 0.6 0.6)
+				(thickness 0.075)
+			)
+			(justify left bottom mirror)
+		)
+	)
+	(gr_text "<-\nRTS\nVID"
+		(at 134.3 92.3 0)
+		(layer "B.SilkS")
+		(effects
+			(font
+				(size 0.6 0.6)
+				(thickness 0.075)
+			)
+			(justify left bottom mirror)
+		)
+	)
+	(gr_text "VCC2"
+		(at 134.8 99.3 -0)
+		(layer "B.SilkS")
+		(effects
+			(font
+				(size 0.6 0.6)
+				(thickness 0.075)
+			)
+			(justify left bottom mirror)
+		)
+	)
+	(gr_text "<-\nRX1\nVOC"
+		(at 150.305 94.9 0)
+		(layer "B.SilkS")
+		(effects
+			(font
+				(size 0.6 0.6)
+				(thickness 0.075)
+			)
+			(justify left bottom mirror)
