File: usb_typec_serial_insulation_adum1412/usb_typec_serial_insulation_adum1412.kicad_pcb (KiCad board)
At the start: 2 copper layers, 27 x 17 mm, 5 parts, among them J1 Conn_01x06_Socket, J2 Conn_01x06_Socket, U1 ADuM1412

Commit message: add rev3.3 zebra 1412
add rev3.3 zebra 1412
Other:
- board text added: "ZEBRA ADuM1412 USB SERIAL ISOLATOR REV 3.3 260911 TSUKUSEI WORKS"
- board text removed: "usb typec serial inslation ADuM1412 V3.2 260430 takurx"
Changed lines of the file:
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@@
 		)
 	)
-	(gr_text "usb typec serial inslation\nADuM1412\nV3.2 260430 takurx"
-		(at 143.1 89.6 90)
+	(gr_text "ZEBRA ADuM1412\nUSB SERIAL ISOLATOR\nREV 3.3 260911\nTSUKUSEI WORKS"
+		(at 144 90 90)
 		(layer "B.SilkS")
 		(effects
